File: swap65.kicad_pcb (KiCad board)
At the start: 2 copper layers, 309.6 x 100 mm, 168 parts, among them J1 USB_C_Receptacle_USB2.0, J2 OLED, J3 DB, SW1 SW_Push, SW10 A, SW11 Z, SW12 LWin, SW13 2, SW14 W, SW15 S, SW16 X, SW17 LAlt, SW18 3, SW19 E, SW2 SW_Push, SW20 D, SW21 C, SW22 4, SW23 R, SW24 F, SW25 V, SW26 5, SW27 T, SW28 G, SW29 B, SW3 Esc, SW30 Space, SW31 6, SW32 Y, SW33 H, SW34 N, SW35 7, SW36 U, SW37 J, SW38 M, SW39 8, SW4 Tab, SW40 I, SW41 K, SW42 Comma, SW43 9, SW44 O, SW45 L, SW46 Period, SW47 RAlt, SW48 0, SW49 P, SW5 Caps, SW50 Colon, SW51 Slash, SW52 Fn, SW53 Minus, SW54 [, SW55 Quote, SW56 Plus, SW57 ], SW58 RShift, SW59 Left, SW6 LShift, SW60 Pipe, SW61 BkSlsh, SW62 Enter, SW63 Up, SW64 Down, SW65 BkSpc, SW66 Tilde, SW67 Right, SW7 LCtrl, SW8 1, SW9 Q, U1 RP2040, U2 SRV05-4, U3 W25Q128JVS, U4 XC6206PxxxMR, Y1 12MHz

Commit message: finalized second pass at routing
Parts:
- moved C16 0.43 mm to (360.2, 136.1)
- moved C1 0.10 mm to (358.4, 129.8)
Routing:
- net COL7: track 245.3 -> 239.6 mm
- net COL8: track 224.9 -> 219.9 mm
- net GND: track 19.6 -> 24.2 mm, vias 26 -> 27
- net COL6: track 261.8 -> 257.5 mm
- net COL11: track 173.7 -> 170.6 mm
- net COL3: track 313.1 -> 311.9 mm
- net COL4: track 297.2 -> 296.1 mm
- net +3V3: track 100.8 -> 101.4 mm
